File: cad/ledui.sch (EAGLE design)
At the start: 18 parts, among them SW1 SWITCH-SPDT, U1 CAP1298

Commit message: tweak
Other:
- moved on the sheet: C10, C8, C9, U1
Changed lines of the file:
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@@
 <part name="VCC1" library="jaw" deviceset="PWR-VCC" device=""/>
 <part name="C7" library="jaw" deviceset="C" device="0603" value="10u"/>
-<part name="FRAME1" library="frames" deviceset="FRAME_B_L" device=""/>
 <part name="SW1" library="jaw" deviceset="SWITCH-SPDT" device=""/>
 <part name="C8" library="jaw" deviceset="C" device="0603" value=".1u"/>
@@
 <part name="U$2" library="adafruit" deviceset="FIDUCIAL" device=""/>
 <part name="U$3" library="jaw" deviceset="ROBOTMAN-LOGO" device=""/>
+<part name="FRAME2" library="frames" deviceset="FRAME_A_L" device=""/>
 </parts>
 <sheets>
@@
 <instance part="VCC1" gate="G$1" x="81.28" y="53.34"/>
 <instance part="C7" gate="G$1" x="73.66" y="48.26" rot="R180"/>
-<instance part="FRAME1" gate="G$1" x="0" y="0"/>
-<instance part="FRAME1" gate="G$2" x="325.12" y="0"/>
 <instance part="SW1" gate="G$1" x="66.04" y="71.12"/>
-<instance part="C8" gate="G$1" x="33.02" y="210.82"/>
-<instance part="VCC2" gate="G$1" x="33.02" y="218.44"/>
-<instance part="GND3" gate="G$1" x="33.02" y="205.74"/>
-<instance part="VCC3" gate="G$1" x="53.34" y="198.12"/>
-<instance part="GND4" gate="G$1" x="53.34" y="170.18"/>
-<instance part="U1" gate="G$1" x="68.58" y="182.88"/>
-<instance part="C9" gate="G$1" x="38.1" y="210.82"/>
-<instance part="C10" gate="G$1" x="27.94" y="210.82"/>
-<instance part="U$1" gate="G$1" x="330.2" y="30.48"/>
-<instance part="U$2" gate="G$1" x="335.28" y="30.48"/>
-<instance part="U$3" gate="G$1" x="419.1" y="27.94"/>
+<instance part="C8" gate="G$1" x="50.8" y="137.16"/>
+<instance part="VCC2" gate="G$1" x="50.8" y="147.32"/>
+<instance part="GND3" gate="G$1" x="50.8" y="132.08"/>
+<instance part="VCC3" gate="G$1" x="71.12" y="142.24"/>
+<instance part="GND4" gate="G$1" x="71.12" y="114.3"/>
+<instance part="U1" gate="G$1" x="86.36" y="127"/>
+<instance part="C9" gate="G$1" x="55.88" y="137.16"/>
+<instance part="C10" gate="G$1" x="45.72" y="137.16"/>
+<instance part="U$1" gate="G$1" x="177.8" y="30.48"/>
+<instance part="U$2" gate="G$1" x="185.42" y="30.48"/>
+<instance part="U$3" gate="G$1" x="266.7" y="27.94"/>
+<instance part="FRAME2" gate="G$1" x="0" y="0"/>
+<instance part="FRAME2" gate="G$2" x="172.72" y="0"/>
 </instances>
 <busses>
@@
 <pinref part="GND3" gate="G$1" pin="GND"/>
 <pinref part="C10" gate="G$1" pin="P$2"/>
-<wire x1="27.94" y1="208.28" x2="33.02" y2="208.28" width="0.1524" layer="91"/>
-<junction x="33.02" y="208.28"/>
+<wire x1="45.72" y1="134.62" x2="50.8" y2="134.62" width="0.1524" layer="91"/>
+<junction x="50.8" y="134.62"/>
 <pinref part="C9" gate="G$1" pin="P$2"/>
-<wire x1="33.02" y1="208.28" x2="38.1" y2="208.28" width="0.1524" layer="91"/>
+<wire x1="50.8" y1="134.62" x2="55.88" y2="134.62" width="0.1524" layer="91"/>
 </segment>
 <segment>
 <pinref part="U1" gate="G$1" pin="GND"/>
 <pinref part="GND4" gate="G$1" pin="GND"/>
-<wire x1="53.34" y1="172.72" x2="53.34" y2="175.26" width="0.1524" layer="91"/>
+<wire x1="71.12" y1="116.84" x2="71.12" y2="119.38" width="0.1524" layer="91"/>
 </segment>
 </net>
@@
 <pinref part="VCC2" gate="G$1" pin="VCC"/>
 <pinref part="C9" gate="G$1" pin="P$1"/>
-<wire x1="33.02" y1="215.9" x2="38.1" y2="215.9" width="0.1524" layer="91"/>
-<junction x="33.02" y="215.9"/>
+<wire x1="50.8" y1="142.24" x2="55.88" y2="142.24" width="0.1524" layer="91"/>
+<junction x="50.8" y="142.24"/>
 <pinref part="C10" gate="G$1" pin="P$1"/>
-<wire x1="27.94" y1="215.9" x2="33.02" y2="215.9" width="0.1524" layer="91"/>
+<wire x1="45.72" y1="142.24" x2="50.8" y2="142.24" width="0.1524" layer="91"/>
+<wire x1="50.8" y1="142.24" x2="50.8" y2="144.78" width="0.1524" layer="91"/>
 </segment>
 <segment>
 <pinref part="U1" gate="G$1" pin="VCC"/>
 <pinref part="VCC3" gate="G$1" pin="VCC"/>
-<wire x1="53.34" y1="195.58" x2="53.34" y2="193.04" width="0.1524" layer="91"/>
+<wire x1="71.12" y1="139.7" x2="71.12" y2="137.16" width="0.1524" layer="91"/>
 </segment>
 </net>
@@
 </segment>
 <segment>
-<label x="43.18" y="180.34" size="1.27" layer="95"/>
+<label x="60.96" y="124.46" size="1.27" layer="95"/>
 <pinref part="U1" gate="G$1" pin="SCL"/>
-<wire x1="53.34" y1="180.34" x2="48.26" y2="180.34" width="0.1524" layer="91"/>
-<junction x="53.34" y="180.34"/>
+<wire x1="71.12" y1="124.46" x2="66.04" y2="124.46" width="0.1524" layer="91"/>
+<junction x="71.12" y="124.46"/>
 </segment>
 </net>
@@
 </segment>
 <segment>
-<label x="43.18" y="182.88" size="1.27" layer="95"/>
+<label x="60.96" y="127" size="1.27" layer="95"/>
 <pinref part="U1" gate="G$1" pin="SDA"/>
-<wire x1="53.34" y1="182.88" x2="48.26" y2="182.88" width="0.1524" layer="91"/>
-<junction x="53.34" y="182.88"/>
+<wire x1="71.12" y1="127" x2="66.04" y2="127" width="0.1524" layer="91"/>
+<junction x="71.12" y="127"/>
 </segment>
 </net>
@@
 <segment>
 <pinref part="U1" gate="G$1" pin="CS1"/>
-<wire x1="83.82" y1="193.04" x2="88.9" y2="193.04" width="0.1524" layer="91"/>
+<wire x1="101.6" y1="137.16" x2="106.68" y2="137.16" width="0.1524" layer="91"/>
 </segment>
 </net>
@@
 <segment>
 <pinref part="U1" gate="G$1" pin="CS2"/>
-<wire x1="83.82" y1="190.5" x2="88.9" y2="190.5" width="0.1524" layer="91"/>
+<wire x1="101.6" y1="134.62" x2="106.68" y2="134.62" width="0.1524" layer="91"/>
 </segment>
 </net>
@@
 <segment>
 <pinref part="U1" gate="G$1" pin="CS3"/>
-<wire x1="83.82" y1="187.96" x2="88.9" y2="187.96" width="0.1524" layer="91"/>
+<wire x1="101.6" y1="132.08" x2="106.68" y2="132.08" width="0.1524" layer="91"/>
 </segment>
 </net>
@@
 <segment>
 <pinref part="U1" gate="G$1" pin="CS4"/>
-<wire x1="83.82" y1="185.42" x2="88.9" y2="185.42" width="0.1524" layer="91"/>
+<wire x1="101.6" y1="129.54" x2="106.68" y2="129.54" width="0.1524" layer="91"/>
 </segment>
 </net>
@@
 <segment>
 <pinref part="U1" gate="G$1" pin="CS5"/>
-<wire x1="83.82" y1="182.88" x2="88.9" y2="182.88" width="0.1524" layer="91"/>
+<wire x1="101.6" y1="127" x2="106.68" y2="127" width="0.1524" layer="91"/>
 </segment>
 </net>
@@
 <segment>
 <pinref part="U1" gate="G$1" pin="CS6"/>
-<wire x1="83.82" y1="180.34" x2="88.9" y2="180.34" width="0.1524" layer="91"/>
+<wire x1="101.6" y1="124.46" x2="106.68" y2="124.46" width="0.1524" layer="91"/>
 </segment>
 </net>
@@
 <segment>
 <pinref part="U1" gate="G$1" pin="CS7"/>
-<wire x1="83.82" y1="177.8" x2="88.9" y2="177.8" width="0.1524" layer="91"/>
+<wire x1="101.6" y1="121.92" x2="106.68" y2="121.92" width="0.1524" layer="91"/>
 </segment>
 </net>
@@
 <segment>
 <pinref part="U1" gate="G$1" pin="CS8"/>
-<wire x1="83.82" y1="175.26" x2="88.9" y2="175.26" width="0.1524" layer="91"/>
-</segment>
-</net>
+<wire x1="101.6" y1="119.38" x2="106.68" y2="119.38" width="0.1524" layer="91"/>
+</segment>
+</net>
