File: cad/ledstick.brd (EAGLE design)
At the start: 475 x 12.5 mm, 31 parts, among them J1 HEADER-4X1-PTH, J2 HEADER-4X1-PTH, U1 BH1745, U4 TMP100, U5 TMP100

Commit message: tweak
Parts:
- C1, C2, C3: value (none) -> .1u
- moved J1 2.00 mm to (141.0, 2.50)
- moved J2 2.00 mm to (50.0, 2.50)
Routing:
- net GND: track 348.6 -> 350.6 mm
- net VCC: track 351.4 -> 353.4 mm
- net SDA: track 335.5 -> 337.5 mm
- net SCL: track 345.0 -> 347.0 mm
- net N$22: track 367.4 -> 369.4 mm
- net N$21: track 372.2 -> 374.2 mm
- net N$20: track 13.8 -> 15.8 mm
- net N$19: track 35.8 -> 37.8 mm
Other:
- board size 475 x 12.5 mm -> 477 x 12.5 mm
- board text added: "Light makes photography. Embrace light. Admire it. Love it. But above all, know light. Know it for all you are worth, and you will know the key to photography. -- George Eastman"

Commit message: initial commit
Connections:
- net GND: now also U1.4
Routing:
- net GND: track 350.6 -> 352.0 mm
Changed lines of the file:
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@@
 <wire x1="329.5" y1="5.45" x2="329.25" y2="5.2" width="0.35" layer="1"/>
 <wire x1="329.25" y1="5.2" x2="328" y2="5.2" width="0.35" layer="1"/>
-<wire x1="331.6" y1="6" x2="330.8" y2="6" width="0.25" layer="1"/>
-<wire x1="330.8" y1="6" x2="330.5" y2="5.7" width="0.25" layer="1"/>
-<wire x1="330.5" y1="5.7" x2="330.25" y2="5.45" width="0.25" layer="1"/>
-<wire x1="330.25" y1="5.45" x2="329.5" y2="5.45" width="0.25" layer="1"/>
+<wire x1="331.6" y1="6" x2="330.6" y2="6" width="0.25" layer="1"/>
 <via x="375.8" y="5.2" extent="1-16" drill="0.35"/>
 <wire x1="374.5" y1="5.45" x2="374.75" y2="5.2" width="0.35" layer="1"/>
@@
 <contactref element="U4" pad="3"/>
 <wire x1="181.85" y1="7.2" x2="181.85" y2="6.25" width="0.3" layer="1"/>
+<contactref element="U1" pad="4"/>
+<wire x1="331.6" y1="5.5" x2="330.4" y2="5.5" width="0.25" layer="1"/>
+<wire x1="330.4" y1="5.5" x2="329.55" y2="5.5" width="0.25" layer="1"/>
+<wire x1="329.55" y1="5.5" x2="329.5" y2="5.45" width="0.25" layer="1"/>
+<wire x1="330.6" y1="6" x2="330.4" y2="5.8" width="0.25" layer="1"/>
+<wire x1="330.4" y1="5.8" x2="330.4" y2="5.5" width="0.25" layer="1"/>
 </signal>
 <signal name="SDA">
