File: cad/ledstick.sch (EAGLE design)
At the start: 31 parts, among them J1 HEADER-4X1-PTH, J2 HEADER-4X1-PTH, U1 BH1745, U4 TMP100, U5 TMP100

Commit message: tweak
Parts:
- C1, C2, C3: value (none) -> .1u
Changed lines of the file:
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@@
 <part name="LED20" library="jaw" deviceset="LED" device="-L4-P1A" value="C"/>
 <part name="U1" library="jaw" deviceset="BH1745" device=""/>
-<part name="C1" library="jaw" deviceset="C" device="0603"/>
+<part name="C1" library="jaw" deviceset="C" device="0603" value=".1u"/>
 <part name="VCC1" library="jaw" deviceset="PWR-VCC" device=""/>
 <part name="GND1" library="jaw" deviceset="PWR-GND" device=""/>
-<part name="C2" library="jaw" deviceset="C" device="0603"/>
-<part name="C3" library="jaw" deviceset="C" device="0603"/>
+<part name="C2" library="jaw" deviceset="C" device="0603" value=".1u"/>
+<part name="C3" library="jaw" deviceset="C" device="0603" value=".1u"/>
 <part name="VCC3" library="jaw" deviceset="PWR-VCC" device=""/>
 <part name="VCC4" library="jaw" deviceset="PWR-VCC" device=""/>

Commit message: initial commit
Connections:
- net GND: now also U1.TEST
Other:
- note added: "addr = 0x72"
- note added: "addr = 0x90"
- note added: "addr = 0x96"
Changed lines of the file:
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@@
 <sheet>
 <plain>
+<text x="68.58" y="68.58" size="2.54" layer="97" ratio="10">addr = 0x90</text>
+<text x="119.38" y="68.58" size="2.54" layer="97" ratio="10">addr = 0x96</text>
+<text x="2.54" y="71.12" size="2.54" layer="97" ratio="10">addr = 0x72</text>
 </plain>
 <instances>
@@
 <label x="73.66" y="83.82" size="1.778" layer="95"/>
 </segment>
-</net>
+<segment>
+<pinref part="U1" gate="G$1" pin="TEST"/>
+<wire x1="15.24" y1="81.28" x2="12.7" y2="81.28" width="0.1524" layer="91"/>
+<label x="10.16" y="81.28" size="1.778" layer="95" ratio="10"/>
+</segment>
+</net>
