File: cad/ledui.brd (EAGLE design)
At the start: 100 x 35 mm, 18 parts, among them SW1 SWITCH-SPDT, U1 CAP1298

Commit message: tweak
Routing:
- net VCC: track 126.2 -> 132.9 mm
- net GND: vias 24 -> 32
Other:
- board text added: "OFF"
- board text added: "ON"
Changed lines of the file:
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@@
 <rectangle x1="13" y1="2.5" x2="45" y2="4" layer="21"/>
 <rectangle x1="45" y1="1" x2="50" y2="4" layer="21"/>
+<text x="9" y="28" size="2" layer="21" ratio="15">ON</text>
+<text x="9" y="22" size="2" layer="21" ratio="15">OFF</text>
 </plain>
 <attributes>
@@
 <attribute name="VALUE" x="28.914" y="7.222" size="1" layer="28" font="vector" ratio="10" rot="MR90"/>
 </element>
-<element name="SW1" library="jaw" package="ALPS-SSAJ120100" value="SWITCH-SPDT" x="7" y="26" rot="R270"/>
+<element name="SW1" library="jaw" package="ALPS-SSAJ120100" value="SWITCH-SPDT" x="7" y="26" smashed="yes" rot="R270">
+<attribute name="NAME" x="5.8" y="21" size="1" layer="25" ratio="10"/>
+</element>
 <element name="C8" library="jaw" package="SMD0603" value=".1u" x="48" y="31.5" smashed="yes" rot="MR180">
 <attribute name="NAME" x="49.078" y="32.616" size="1" layer="26" font="vector" ratio="10" rot="MR0"/>
@@
 <via x="12.1" y="32" extent="1-16" drill="0.35"/>
 <via x="13.1" y="5" extent="1-16" drill="0.35"/>
-<via x="21.1" y="4" extent="1-16" drill="0.35"/>
+<via x="21.2" y="5" extent="1-16" drill="0.35"/>
 <via x="21" y="32" extent="1-16" drill="0.35"/>
 <via x="33" y="32" extent="1-16" drill="0.35"/>
@@
 <via x="48.4" y="27.6" extent="1-16" drill="0.35"/>
 <via x="47.6" y="27.6" extent="1-16" drill="0.35"/>
-<wire x1="48" y1="28" x2="47.6" y2="27.6" width="0" layer="19" extent="16-16"/>
+<via x="16.5" y="22.9" extent="1-16" drill="0.35"/>
+<via x="21" y="17" extent="1-16" drill="0.35"/>
+<via x="26" y="20.9" extent="1-16" drill="0.35"/>
+<via x="29.4" y="17" extent="1-16" drill="0.35"/>
+<via x="37" y="22" extent="1-16" drill="0.35"/>
+<via x="26" y="12.3" extent="1-16" drill="0.35"/>
+<via x="29.5" y="13" extent="1-16" drill="0.35"/>
+<via x="23" y="8" extent="1-16" drill="0.35"/>
 </signal>
 <signal name="VCC">
@@
 <contactref element="C7" pad="2"/>
 <contactref element="C8" pad="1"/>
-<wire x1="31.2" y1="27.5" x2="31.2" y2="15" width="0.25" layer="16"/>
+<wire x1="31.2" y1="27.5" x2="31.2" y2="22.6" width="0.25" layer="16"/>
+<wire x1="31.2" y1="22.6" x2="31.2" y2="15" width="0.25" layer="16"/>
 <wire x1="31.2" y1="15" x2="31.2" y2="10" width="0.25" layer="16"/>
 <wire x1="31.2" y1="10" x2="31" y2="9.8" width="0.25" layer="16"/>
@@
 <wire x1="96.8" y1="7.2" x2="96.05" y2="6.45" width="0.25" layer="16"/>
 <wire x1="40.2" y1="26" x2="38.9" y2="26" width="0.25" layer="16"/>
-<wire x1="31.2" y1="27.5" x2="33.3" y2="27.5" width="0" layer="19" extent="16-16"/>
+<wire x1="33.3" y1="27.5" x2="33.3" y2="23" width="0.25" layer="16"/>
+<wire x1="33.3" y1="23" x2="32.9" y2="22.6" width="0.25" layer="16"/>
+<wire x1="32.9" y1="22.6" x2="31.2" y2="22.6" width="0.25" layer="16"/>
 </signal>
 <signal name="S$4">
