File: cad/ledcontrol.brd (EAGLE design)
At the start: 100 x 35 mm, 85 parts, among them CN1 HEADER-3X2-PTH, CN3 HEADER-1X2-THM, J1 HEADER-4X1-PTH, J2 HEADER-4X1-PTH, Q1 IRLML6344TRPBF, Q2 MOSFET-P, Q3 MOSFETSOT-23, Q4 ZXMN6A08GTA, Q5 ZXMN6A08GTA, Q6 IRLML6344TRPBF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

Commit message: .
Parts:
- removed U$3: SYMBOL-WARNING, jaw:SYMBOL-WARNING
- added C25, C26: 10u,12V, jaw:SMD0603
- added C27: .1u,12V, jaw:SMD0603
- C1: value 1u, 12V -> .1u, 12V
Connections:
- net GND: now also C25.2, C26.2, C27.2
- net VCCM: now also C25.1, C26.1, C27.1
Routing:
- net GND: track 135.9 -> 142.2 mm, vias 36 -> 66
- net ADCVBAT: track 28.3 -> 30.1 mm
- net L0M: track 77.5 -> 79.3 mm
- net VCCM: track 172.5 -> 174.1 mm
- added copper zone on layer 15, net GND

Commit message: tweak
Parts:
- D3, D4: value PMEG6020ETR115 -> ss3p6; device jaw:DO-214AC -> jaw:DO-220AA
- R15, R23: value 88k7 -> 88k7, .1%
- R16, R18, R24: value 3k3 -> 3k3, .1%
- R17: value 14k7 -> 14k7, .1%
- U2: value LMP8640 -> LMP8640-H
- VREG1: value MCP1824 -> MCP1754
- moved C13 8.25 mm to (80.0, 8.00), turned to 90 degrees
- moved R14 6.32 mm to (73.0, 8.00), turned to 270 degrees
- moved U2 2.83 mm to (77.0, 8.00), turned to 270 degrees
- moved LED1 0.40 mm to (7.40, 25.0)
- moved R8 0.40 mm to (7.40, 27.0)
- turned D3 to 180 degrees
- turned D4 to 180 degrees
Connections:
- net VCC: no longer CN3.P$1, D5.C
- net VCCM: now also CN3.P$1, D5.C
Routing:
- net VCCM: track 174.1 -> 202.8 mm, vias 2 -> 3
- net VCC: track 52.7 -> 48.6 mm
- net N$16: track 33.8 -> 37.3 mm
- net L0P: track 31.3 -> 32.7 mm
- net L1P: track 30.8 -> 32.2 mm
- net IOLED: track 31.0 -> 30.4 mm
- net SPIMISO: track 21.4 -> 20.9 mm
- net L0M: track 79.3 -> 78.8 mm
- net GND: vias 66 -> 65
- added copper zone on layer 1, net N$22
- added copper zone on layer 1, net N$23
Other:
- board text added: "I hate the day, because it lendeth light To see all things, but not my love to see. -- Edmund Spenser"
- board text added: "INPUT: 12V MAX"
- board text added: "Light-Stick"
- board text removed: "INPUT: 6V MAX"
- board text removed: "Lighty-Light"
- board text removed: "WARNING: HIGH VOLTAGE!"

Commit message: initial commit
Connections:
- net GND: now also J2.P$1; no longer J2.P$4
- net VCC: now also J2.P$4; no longer J2.P$1
Routing:
- net VCC: track 48.6 -> 46.4 mm, vias 12 -> 13

Commit message: more power
Parts:
- added C28, C29: 10u,12V, jaw:SMD0603
- added D6: DIODESOD-323, jaw:SOD-323
- added L4, L5: (no value), jaw:SRR1260
- D3, D4: device jaw:DO-220AA -> jaw:DO-214AC
- L2, L3: value 220u -> 22u; device jaw:SRR1260 -> jaw:BOURNS2303
- Q2: device jaw:SOT-23-3 -> jaw:SOT-23-3@1
- Q4, Q5: value ZXMN6A08GTA -> AON6246; device jaw:SOT223 -> jaw:DFN5X6-8LEP1
- moved L2 1.00 mm to (63.5, 8.50), turned to 240 degrees
- moved L3 1.00 mm to (63.5, 26.5), turned to 60 degrees
- moved Q4 1.00 mm to (50.0, 10.0), turned to 90 degrees
- moved Q5 1.00 mm to (50.0, 28.0), turned to 90 degrees
- moved C1 0.10 mm to (43.0, 3.50)
- moved C25 0.10 mm to (41.5, 3.50)
- moved Q3 0.10 mm to (30.6, 9.00), turned to 180 degrees
- turned Q1 to 90 degrees
- turned Q6 to 0 degrees
Connections:
- new net VIN: C1.1, C25.1, D6.C, Q2.2, R11.2, VREG1.1
- net GND: now also C28.2, C29.2
- net L0M: now also Q4.P$1, Q4.P$2, Q4.P$3; no longer Q4.3
- net L1M: now also Q5.P$1, Q5.P$2, Q5.P$3; no longer Q5.3
- net N$12: now also L5.P$1, Q5.P$5, Q5.P$6, Q5.P$7, Q5.P$8, Q5.P$9; no longer Q5.2, Q5.4
- net N$15: now also Q5.P$4; no longer Q5.1
- net N$2: now also L4.P$1, Q4.P$5, Q4.P$6, Q4.P$7, Q4.P$8, Q4.P$9; no longer Q4.2, Q4.4
- net N$6: now also Q4.P$4; no longer Q4.1
- net VCCM: now also C28.1, C29.1, D6.A, L4.P$2, L5.P$2; no longer C1.1, C25.1, Q2.2, R11.2, VREG1.1
Routing:
- net VIN: track 0.00 -> 16.9 mm, vias 0 -> 2
- net N$12: track 37.2 -> 50.5 mm, vias 0 -> 2
- net N$6: track 13.6 -> 21.9 mm, vias 0 -> 2
- net VCCM: track 202.8 -> 210.3 mm
- net N$2: track 35.6 -> 40.1 mm
- net GND: track 142.2 -> 146.6 mm
- net L1M: track 83.8 -> 87.9 mm
- net L0M: track 78.8 -> 80.7 mm
- net N$15: track 22.7 -> 21.6 mm
- net L1P: track 32.2 -> 31.3 mm
Other:
- board text added: "JAW 2015-07"
- board text added: "LEDCTL Rev. 1"
- board text removed: "I hate the day, because it lendeth light To see all things, but not my love to see. -- Edmund Spenser"
- board text removed: "LEDCTL Rev. 0"

Commit message: tweak
Parts:
- C1: value .1u, 12V -> .1u, 16V
- C11, C5: value .002u -> .002u,100V
- C25, C26, C28, C29: value 10u,12V -> 10u,16V
- C27: value .1u,12V -> .1u,16V
Changed lines of the file:
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@@
 <layer number="3" name="Route3" color="4" fill="3" visible="no" active="no"/>
 <layer number="14" name="Route14" color="1" fill="6" visible="no" active="no"/>
-<layer number="15" name="Route15" color="1" fill="1" visible="yes" active="yes"/>
+<layer number="15" name="Route15" color="1" fill="1" visible="no" active="yes"/>
 <layer number="16" name="Bottom" color="6" fill="1" visible="no" active="yes"/>
 <layer number="17" name="Pads" color="2" fill="1" visible="yes" active="yes"/>
@@
 </autorouter>
 <elements>
-<element name="C1" library="jaw" package="SMD0603" value=".1u, 12V" x="43" y="3.5" smashed="yes" rot="R90">
+<element name="C1" library="jaw" package="SMD0603" value=".1u, 16V" x="43" y="3.5" smashed="yes" rot="R90">
 <attribute name="NAME" x="43.322" y="1.016" size="1" layer="25" font="vector" ratio="10"/>
 <attribute name="VALUE" x="43.486" y="0.722" size="1" layer="27" font="vector" ratio="10" rot="R90"/>
@@
 <attribute name="VALUE" x="16.478" y="25.886" size="1" layer="27" font="vector" ratio="10" rot="R180"/>
 </element>
-<element name="C11" library="jaw" package="SMD0603" value=".002u" x="55" y="26" smashed="yes" rot="R270">
+<element name="C11" library="jaw" package="SMD0603" value=".002u,100V" x="55" y="26" smashed="yes" rot="R270">
 <attribute name="NAME" x="55.916" y="27.278" size="1" layer="25" font="vector" ratio="10" rot="R270"/>
 <attribute name="VALUE" x="54.822" y="25.314" size="1" layer="27" font="vector" ratio="10"/>
@@
 <attribute name="VALUE" x="28.414" y="19.478" size="1" layer="27" font="vector" ratio="10" rot="R270"/>
 </element>
-<element name="C5" library="jaw" package="SMD0603" value=".002u" x="55" y="9.5" smashed="yes" rot="R270">
+<element name="C5" library="jaw" package="SMD0603" value=".002u,100V" x="55" y="9.5" smashed="yes" rot="R270">
 <attribute name="NAME" x="56.016" y="10.578" size="1" layer="25" font="vector" ratio="10" rot="R270"/>
 <attribute name="VALUE" x="54.722" y="8.714" size="1" layer="27" font="vector" ratio="10"/>
@@
 <attribute name="VALUE" x="36.4" y="15.3" size="0.5" layer="27" rot="R180"/>
 </element>
-<element name="C25" library="jaw" package="SMD0603" value="10u,12V" x="41.5" y="3.5" smashed="yes" rot="R90">
+<element name="C25" library="jaw" package="SMD0603" value="10u,16V" x="41.5" y="3.5" smashed="yes" rot="R90">
 <attribute name="NAME" x="40.222" y="1.016" size="1" layer="25" font="vector" ratio="10"/>
 <attribute name="VALUE" x="41.886" y="1.022" size="1" layer="27" font="vector" ratio="10" rot="R90"/>
 </element>
-<element name="C26" library="jaw" package="SMD0603" value="10u,12V" x="102" y="9.5" smashed="yes">
+<element name="C26" library="jaw" package="SMD0603" value="10u,16V" x="102" y="9.5" smashed="yes">
 <attribute name="NAME" x="100.278" y="9.984" size="1" layer="25" font="vector" ratio="10" rot="R180"/>
 <attribute name="VALUE" x="100.222" y="7.414" size="1" layer="27" font="vector" ratio="10"/>
 </element>
-<element name="C27" library="jaw" package="SMD0603" value=".1u,12V" x="102" y="8" smashed="yes">
+<element name="C27" library="jaw" package="SMD0603" value=".1u,16V" x="102" y="8" smashed="yes">
 <attribute name="NAME" x="100.178" y="8.484" size="1" layer="25" font="vector" ratio="10" rot="R180"/>
 <attribute name="VALUE" x="100.222" y="5.914" size="1" layer="27" font="vector" ratio="10"/>
 </element>
 <element name="D6" library="jaw" package="SOD-323" value="DIODESOD-323" x="44.6" y="3.5" rot="R90"/>
-<element name="C28" library="jaw" package="SMD0603" value="10u,12V" x="75" y="31"/>
-<element name="C29" library="jaw" package="SMD0603" value="10u,12V" x="77" y="4" rot="R180"/>
+<element name="C28" library="jaw" package="SMD0603" value="10u,16V" x="75" y="31"/>
+<element name="C29" library="jaw" package="SMD0603" value="10u,16V" x="77" y="4" rot="R180"/>
 <element name="L4" library="jaw" package="SRR1260" value="" x="63.5" y="9.5" rot="R270"/>
 <element name="L5" library="jaw" package="SRR1260" value="" x="63.5" y="25.5" rot="R90"/>
@@
 <wire x1="72.55" y1="28.35" x2="72" y2="27.8" width="0.3" layer="1"/>
 <via x="34" y="2" extent="1-16" drill="0.5"/>
-<wire x1="36.7" y1="2.05" x2="34.05" y2="2.05" width="0.5" layer="1"/>
 <wire x1="34.05" y1="2.05" x2="34" y2="2" width="0.5" layer="1"/>
 <wire x1="32.5" y1="2.7" x2="33.3" y2="2.7" width="0.5" layer="1"/>
@@
 <via x="6.3" y="12.1" extent="1-16" drill="0.35"/>
 <wire x1="6.3" y1="11" x2="6.3" y2="12.1" width="0.25" layer="1"/>
+<wire x1="36.7" y1="2.05" x2="34.05" y2="2.05" width="0.5" layer="1"/>
 <wire x1="25" y1="13.3" x2="24.2" y2="13.3" width="0" layer="19" extent="1-1"/>
 </signal>
@@
 <wire x1="50.001" y1="10.201" x2="50" y2="10" width="1.5" layer="1"/>
 <wire x1="71.6" y1="14.5" x2="66.7" y2="14.5" width="2" layer="1"/>
-<wire x1="66.7" y1="14.5" x2="50.301" y2="14.5" width="2" layer="1"/>
+<wire x1="66.7" y1="14.5" x2="63.6" y2="14.5" width="2" layer="1"/>
+<wire x1="63.6" y1="14.5" x2="50.301" y2="14.5" width="2" layer="1"/>
 <wire x1="50.301" y1="14.5" x2="50.001" y2="14.2" width="2" layer="1"/>
 <wire x1="66.75" y1="14.1291625" x2="66.75" y2="14.45" width="2" layer="1"/>
 <wire x1="66.75" y1="14.45" x2="66.7" y2="14.5" width="2" layer="1"/>
 <contactref element="L4" pad="P$1"/>
-<wire x1="49.1" y1="10.7" x2="49.1" y2="11.9" width="0" layer="19" extent="1-1"/>
-<wire x1="50.001" y1="10.201" x2="49.1" y2="10.7" width="0" layer="19" extent="1-1"/>
-<wire x1="49" y1="9.5" x2="50" y2="10" width="0" layer="19" extent="1-1"/>
-<wire x1="48.895" y1="8.095" x2="48.865" y2="9.365" width="0" layer="19" extent="1-1"/>
-<wire x1="63.5" y1="14.3" x2="47.25" y2="8.095" width="0" layer="19" extent="1-1"/>
+<wire x1="63.5" y1="14.3" x2="63.5" y2="14.4" width="2" layer="1"/>
+<wire x1="63.5" y1="14.4" x2="63.6" y2="14.5" width="2" layer="1"/>
 </signal>
 <signal name="L1P">
@@
 <wire x1="49.9" y1="20.7" x2="49.9" y2="27.9" width="1.5" layer="1"/>
 <wire x1="49.9" y1="27.9" x2="50" y2="28" width="1.5" layer="1"/>
-<wire x1="71.6" y1="20.5" x2="60.2" y2="20.5" width="2" layer="1"/>
+<wire x1="71.6" y1="20.5" x2="63.7" y2="20.5" width="2" layer="1"/>
+<wire x1="63.7" y1="20.5" x2="60.2" y2="20.5" width="2" layer="1"/>
 <wire x1="60.2" y1="20.5" x2="50.1" y2="20.5" width="2" layer="1"/>
 <wire x1="50.1" y1="20.5" x2="49.9" y2="20.7" width="2" layer="1"/>
@@
 <wire x1="60.25" y1="20.55" x2="60.2" y2="20.5" width="2" layer="1"/>
 <contactref element="L5" pad="P$1"/>
-<wire x1="48.965" y1="28.635" x2="48.905" y2="29.905" width="0" layer="19" extent="1-1"/>
-<wire x1="49.9" y1="27.9" x2="49" y2="28.6" width="0" layer="19" extent="1-1"/>
-<wire x1="49" y1="27.4" x2="49.9" y2="27.9" width="0" layer="19" extent="1-1"/>
-<wire x1="49" y1="26.2" x2="48.965" y2="27.365" width="0" layer="19" extent="1-1"/>
-<wire x1="63.5" y1="20.7" x2="47.25" y2="26.095" width="0" layer="19" extent="1-1"/>
+<wire x1="63.5" y1="20.7" x2="63.7" y2="20.5" width="2" layer="1"/>
 </signal>
 <signal name="N$13">

Commit message: more power
Parts:
- added FID1: FIDUCIALUFIDUCIAL, SparkFun-Aesthetics:MICRO-FIDUCIAL
- moved L2 1.03 mm to (64.5, 8.75), turned to 270 degrees
- moved L3 1.03 mm to (62.5, 26.2), turned to 90 degrees
Routing:
- net VCCM: track 210.3 -> 427.2 mm, vias 3 -> 13
- net N$12: track 50.8 -> 58.4 mm, vias 2 -> 6
- net N$2: track 40.4 -> 45.0 mm, vias 0 -> 4
- net ADCBV0: track 58.9 -> 63.1 mm, vias 0 -> 2
- net ADCBV1: track 59.9 -> 63.0 mm, vias 0 -> 2
- net GND: vias 65 -> 66
- added copper zone on layer 16, net N$12
- added copper zone on layer 16, net N$2
Other:
- board text added: "L"
- board text removed: "JAW 2015-06"
- board text removed: "Light-Stick"
