File: cad/ledcontrol.sch (EAGLE design)
At the start: 85 parts, among them CN1 HEADER-3X2-PTH, CN3 HEADER-1X2-THM, J1 HEADER-4X1-PTH, J2 HEADER-4X1-PTH, Q1 IRLML6344TRPBF, Q2 MOSFET-P, Q3 MOSFETSOT-23, Q4 ZXMN6A08GTA, Q5 ZXMN6A08GTA, Q6 IRLML6344TRPBF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

Commit message: .
Parts:
- removed U$3: SYMBOL-WARNING, jaw:SYMBOL-WARNING
- added C25, C26: 10u,12V, jaw:C0603
- added C27: .1u,12V, jaw:C0603
- C1: value 1u, 12V -> .1u, 12V
Connections:
- net GND: now also C25.P$2, C26.P$2, C27.P$2
- net VCCM: now also C25.P$1, C26.P$1, C27.P$1
Other:
- moved on the sheet: VREG1
Changed lines of the file:
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@@
 <part name="VCCM3" library="jaw" deviceset="PWR-VCCM" device=""/>
 <part name="VCC4" library="jaw" deviceset="PWR-VCC" device=""/>
-<part name="C1" library="jaw" deviceset="C" device="0603" value="1u, 12V"/>
+<part name="C1" library="jaw" deviceset="C" device="0603" value=".1u, 12V"/>
 <part name="C2" library="jaw" deviceset="C" device="0603" value="1u"/>
 <part name="C3" library="jaw" deviceset="C" device="1210" value="100u"/>
@@
 <part name="R28" library="jaw" deviceset="R" device="0603" value="1M"/>
 <part name="CN3" library="jaw" deviceset="HEADER-1X2" device="-THM" value="HEADER-1X2-THM"/>
-<part name="U$3" library="jaw" deviceset="SYMBOL-WARNING" device=""/>
 <part name="LOGO1" library="SparkFun-Aesthetics" deviceset="OSHW-LOGO" device="S"/>
 <part name="C24" library="jaw" deviceset="C" device="0603" value=".1u"/>
@@
 <part name="GND23" library="jaw" deviceset="PWR-GND" device=""/>
 <part name="GND24" library="jaw" deviceset="PWR-GND" device=""/>
+<part name="C25" library="jaw" deviceset="C" device="0603" value="10u,12V"/>
+<part name="C26" library="jaw" deviceset="C" device="0603" value="10u,12V"/>
+<part name="C27" library="jaw" deviceset="C" device="0603" value=".1u,12V"/>
+<part name="VCCM7" library="jaw" deviceset="PWR-VCCM" device=""/>
+<part name="GND27" library="jaw" deviceset="PWR-GND" device=""/>
 </parts>
 <sheets>
@@
 <instance part="R10" gate="G$1" x="203.2" y="200.66" rot="R270"/>
 <instance part="CONN1" gate="G$1" x="213.36" y="144.78"/>
-<instance part="VREG1" gate="G$1" x="48.26" y="17.78"/>
+<instance part="VREG1" gate="G$1" x="53.34" y="17.78"/>
 <instance part="Q2" gate="G$1" x="60.96" y="58.42" rot="R180"/>
 <instance part="D2" gate="G$1" x="50.8" y="50.8"/>
@@
 <instance part="R28" gate="G$1" x="149.86" y="20.32" rot="R270"/>
 <instance part="CN3" gate="G$1" x="162.56" y="40.64"/>
-<instance part="U$3" gate="G$1" x="419.1" y="30.48"/>
 <instance part="LOGO1" gate="G$1" x="406.4" y="27.94"/>
 <instance part="C24" gate="G$1" x="187.96" y="22.86"/>
@@
 <instance part="GND23" gate="G$1" x="187.96" y="12.7"/>
 <instance part="GND24" gate="G$1" x="218.44" y="5.08"/>
+<instance part="C25" gate="G$1" x="22.86" y="15.24"/>
+<instance part="C26" gate="G$1" x="370.84" y="243.84"/>
+<instance part="C27" gate="G$1" x="381" y="243.84"/>
+<instance part="VCCM7" gate="G$1" x="375.92" y="254"/>
+<instance part="GND27" gate="G$1" x="375.92" y="233.68"/>
 </instances>
 <busses>
@@
 <pinref part="C1" gate="G$1" pin="P$2"/>
 <pinref part="VREG1" gate="G$1" pin="GND"/>
-<wire x1="17.78" y1="10.16" x2="43.18" y2="10.16" width="0.1524" layer="91"/>
+<wire x1="17.78" y1="10.16" x2="22.86" y2="10.16" width="0.1524" layer="91"/>
 <pinref part="C2" gate="G$1" pin="P$2"/>
-<wire x1="43.18" y1="10.16" x2="48.26" y2="10.16" width="0.1524" layer="91"/>
-<wire x1="48.26" y1="10.16" x2="71.12" y2="10.16" width="0.1524" layer="91"/>
+<wire x1="22.86" y1="10.16" x2="43.18" y2="10.16" width="0.1524" layer="91"/>
+<wire x1="43.18" y1="10.16" x2="53.34" y2="10.16" width="0.1524" layer="91"/>
+<wire x1="53.34" y1="10.16" x2="71.12" y2="10.16" width="0.1524" layer="91"/>
 <wire x1="71.12" y1="10.16" x2="71.12" y2="12.7" width="0.1524" layer="91"/>
-<junction x="48.26" y="10.16"/>
+<junction x="53.34" y="10.16"/>
 <pinref part="C3" gate="G$1" pin="P$2"/>
 <wire x1="71.12" y1="10.16" x2="76.2" y2="10.16" width="0.1524" layer="91"/>
@@
 <wire x1="10.16" y1="10.16" x2="17.78" y2="10.16" width="0.1524" layer="91"/>
 <junction x="17.78" y="10.16"/>
+<pinref part="C25" gate="G$1" pin="P$2"/>
+<wire x1="22.86" y1="12.7" x2="22.86" y2="10.16" width="0.1524" layer="91"/>
+<junction x="22.86" y="10.16"/>
 </segment>
 <segment>
@@
 <wire x1="203.2" y1="25.4" x2="200.66" y2="25.4" width="0.1524" layer="91"/>
 <label x="195.58" y="25.4" size="1.778" layer="95"/>
+</segment>
+<segment>
+<pinref part="C26" gate="G$1" pin="P$2"/>
+<pinref part="C27" gate="G$1" pin="P$2"/>
+<wire x1="370.84" y1="241.3" x2="375.92" y2="241.3" width="0.1524" layer="91"/>
+<pinref part="GND27" gate="G$1" pin="GND"/>
+<wire x1="375.92" y1="241.3" x2="381" y2="241.3" width="0.1524" layer="91"/>
+<wire x1="375.92" y1="241.3" x2="375.92" y2="236.22" width="0.1524" layer="91"/>
+<junction x="375.92" y="241.3"/>
 </segment>
 </net>
@@
 <pinref part="VREG1" gate="G$1" pin="VOUT"/>
 <pinref part="C2" gate="G$1" pin="P$1"/>
-<wire x1="63.5" y1="20.32" x2="71.12" y2="20.32" width="0.1524" layer="91"/>
+<wire x1="68.58" y1="20.32" x2="71.12" y2="20.32" width="0.1524" layer="91"/>
 <pinref part="C3" gate="G$1" pin="P$1"/>
 <wire x1="71.12" y1="20.32" x2="73.66" y2="20.32" width="0.1524" layer="91"/>
@@
 <wire x1="10.16" y1="20.32" x2="17.78" y2="20.32" width="0.1524" layer="91"/>
 <pinref part="C1" gate="G$1" pin="P$1"/>
-<wire x1="17.78" y1="20.32" x2="33.02" y2="20.32" width="0.1524" layer="91"/>
+<wire x1="17.78" y1="20.32" x2="22.86" y2="20.32" width="0.1524" layer="91"/>
+<wire x1="22.86" y1="20.32" x2="38.1" y2="20.32" width="0.1524" layer="91"/>
 <wire x1="17.78" y1="17.78" x2="17.78" y2="20.32" width="0.1524" layer="91"/>
 <junction x="17.78" y="20.32"/>
@@
 <wire x1="10.16" y1="15.24" x2="10.16" y2="20.32" width="0.1524" layer="91"/>
 <junction x="10.16" y="20.32"/>
+<pinref part="C25" gate="G$1" pin="P$1"/>
+<junction x="22.86" y="20.32"/>
 </segment>
 <segment>
@@
 <wire x1="220.98" y1="144.78" x2="223.52" y2="144.78" width="0.1524" layer="91"/>
 <label x="223.52" y="144.78" size="1.27" layer="95"/>
+</segment>
+<segment>
+<pinref part="C26" gate="G$1" pin="P$1"/>
+<pinref part="C27" gate="G$1" pin="P$1"/>
+<wire x1="370.84" y1="248.92" x2="375.92" y2="248.92" width="0.1524" layer="91"/>
+<pinref part="VCCM7" gate="G$1" pin="VCCM"/>
+<wire x1="375.92" y1="248.92" x2="381" y2="248.92" width="0.1524" layer="91"/>
+<wire x1="375.92" y1="248.92" x2="375.92" y2="251.46" width="0.1524" layer="91"/>
+<junction x="375.92" y="248.92"/>
 </segment>
 </net>
@@
 <segment>
 <pinref part="VREG1" gate="G$1" pin="NSHTDN"/>
-<wire x1="33.02" y1="17.78" x2="27.94" y2="17.78" width="0.1524" layer="91"/>
-<label x="20.32" y="17.78" size="1.778" layer="95"/>
-</segment>
-</net>
+<wire x1="38.1" y1="17.78" x2="35.56" y2="17.78" width="0.1524" layer="91"/>
+<label x="27.94" y="17.78" size="1.778" layer="95"/>
+</segment>
+</net>

Commit message: tweak
Parts:
- D3, D4: value PMEG6020ETR115 -> ss3p6; device jaw:DIODEDO-214AC -> jaw:DIODE-DO220AA
- R15, R23: value 88k7 -> 88k7, .1%
- R16, R18, R24: value 3k3 -> 3k3, .1%
- R17: value 14k7 -> 14k7, .1%
- U2: value LMP8640 -> LMP8640-H
- VREG1: value MCP1824 -> MCP1754
Connections:
- net VCC: no longer CN3.P$1, D5.C
- net VCCM: now also CN3.P$1, D5.C
Other:
- note added: "12V max"
- note removed: "6V max"
Changed lines of the file:
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@@
 <part name="R10" library="jaw" deviceset="R" device="0603" value="1M"/>
 <part name="CONN1" library="jaw" deviceset="HEADER-6X2" device="-PTH"/>
-<part name="VREG1" library="jaw" deviceset="MCP1824" device=""/>
+<part name="VREG1" library="jaw" deviceset="MCP1824" device="" value="MCP1754"/>
 <part name="Q2" library="jaw" deviceset="MOSFET-P" device=""/>
 <part name="D2" library="jaw" deviceset="DIODE" device="SOD-323"/>
@@
 <part name="R14" library="jaw" deviceset="R" device="1206" value=".01"/>
 <part name="C5" library="jaw" deviceset="C" device="0603" value=".002u"/>
-<part name="R15" library="jaw" deviceset="R" device="0603" value="88k7"/>
-<part name="R16" library="jaw" deviceset="R" device="0603" value="3k3"/>
+<part name="R15" library="jaw" deviceset="R" device="0603" value="88k7, .1%"/>
+<part name="R16" library="jaw" deviceset="R" device="0603" value="3k3, .1%"/>
 <part name="J1" library="jaw" deviceset="HEADER-4X1" device="-PTH"/>
 <part name="VCCM4" library="jaw" deviceset="PWR-VCCM" device=""/>
-<part name="D3" library="jaw" deviceset="DIODE" device="DO-214AC" value="PMEG6020ETR115"/>
+<part name="D3" library="jaw" deviceset="DIODE" device="-DO220AA" value="ss3p6"/>
 <part name="C6" library="jaw" deviceset="C-POL" device="-KE0" value="100u,100v"/>
 <part name="GND5" library="jaw" deviceset="PWR-GND" device=""/>
 <part name="GND6" library="jaw" deviceset="PWR-GND" device=""/>
-<part name="U2" library="jaw" deviceset="LMP8640" device=""/>
+<part name="U2" library="jaw" deviceset="LMP8640" device="" value="LMP8640-H"/>
 <part name="VCC1" library="jaw" deviceset="PWR-VCC" device=""/>
 <part name="GND11" library="jaw" deviceset="PWR-GND" device=""/>
 <part name="C8" library="jaw" deviceset="C" device="0603" value=".1u"/>
 <part name="C9" library="jaw" deviceset="C" device="0805" value=".1u, 100v"/>
-<part name="R17" library="jaw" deviceset="R" device="0603" value="14k7"/>
-<part name="R18" library="jaw" deviceset="R" device="0603" value="3k3"/>
+<part name="R17" library="jaw" deviceset="R" device="0603" value="14k7, .1%"/>
+<part name="R18" library="jaw" deviceset="R" device="0603" value="3k3, .1%"/>
 <part name="GND12" library="jaw" deviceset="PWR-GND" device=""/>
 <part name="VCCM5" library="jaw" deviceset="PWR-VCCM" device=""/>
@@
 <part name="R22" library="jaw" deviceset="R" device="1206" value=".01"/>
 <part name="C11" library="jaw" deviceset="C" device="0603" value=".002u"/>
-<part name="R23" library="jaw" deviceset="R" device="0603" value="88k7"/>
-<part name="R24" library="jaw" deviceset="R" device="0603" value="3k3"/>
+<part name="R23" library="jaw" deviceset="R" device="0603" value="88k7, .1%"/>
+<part name="R24" library="jaw" deviceset="R" device="0603" value="3k3, .1%"/>
 <part name="VCCM6" library="jaw" deviceset="PWR-VCCM" device=""/>
-<part name="D4" library="jaw" deviceset="DIODE" device="DO-214AC" value="PMEG6020ETR115"/>
+<part name="D4" library="jaw" deviceset="DIODE" device="-DO220AA" value="ss3p6"/>
 <part name="C12" library="jaw" deviceset="C-POL" device="-KE0" value="100u,100v"/>
 <part name="GND13" library="jaw" deviceset="PWR-GND" device=""/>
@@
 <part name="C18" library="jaw" deviceset="C" device="0603" value="1u"/>
 <part name="D5" library="jaw" deviceset="DIODE" device="SOD-323" value="any"/>
-<part name="VCC6" library="jaw" deviceset="PWR-VCC" device=""/>
 <part name="GND22" library="jaw" deviceset="PWR-GND" device=""/>
 <part name="Q6" library="jaw" deviceset="MOSFET" device="SOT-23" value="IRLML6344TRPBF"/>
@@
 <part name="VCCM7" library="jaw" deviceset="PWR-VCCM" device=""/>
 <part name="GND27" library="jaw" deviceset="PWR-GND" device=""/>
+<part name="VCCM8" library="jaw" deviceset="PWR-VCCM" device=""/>
 </parts>
 <sheets>
@@
 <text x="43.18" y="68.58" size="1.778" layer="97">connector
 to switch</text>
-<text x="22.86" y="22.86" size="1.778" layer="97">6V max</text>
+<text x="22.86" y="22.86" size="1.778" layer="97">12V max</text>
 <text x="208.28" y="165.1" size="1.778" layer="97">display</text>
 <text x="208.28" y="134.62" size="1.778" layer="97">programming</text>
@@
 <instance part="C18" gate="G$1" x="271.78" y="96.52"/>
 <instance part="D5" gate="G$1" x="149.86" y="40.64" rot="R90"/>
-<instance part="VCC6" gate="G$1" x="157.48" y="53.34"/>
 <instance part="GND22" gate="G$1" x="157.48" y="12.7"/>
 <instance part="Q6" gate="G$1" x="157.48" y="27.94"/>
@@
 <instance part="VCCM7" gate="G$1" x="375.92" y="254"/>
 <instance part="GND27" gate="G$1" x="375.92" y="233.68"/>
+<instance part="VCCM8" gate="G$1" x="157.48" y="53.34"/>
 </instances>
 <busses>
@@
 </segment>
 <segment>
-<pinref part="VCC6" gate="G$1" pin="VCC"/>
-<wire x1="157.48" y1="50.8" x2="157.48" y2="48.26" width="0.1524" layer="91"/>
-<pinref part="D5" gate="G$1" pin="C"/>
-<wire x1="149.86" y1="43.18" x2="149.86" y2="48.26" width="0.1524" layer="91"/>
-<wire x1="149.86" y1="48.26" x2="157.48" y2="48.26" width="0.1524" layer="91"/>
-<pinref part="CN3" gate="G$1" pin="P$1"/>
-<wire x1="157.48" y1="43.18" x2="157.48" y2="48.26" width="0.1524" layer="91"/>
-<junction x="157.48" y="48.26"/>
-</segment>
-<segment>
 <pinref part="C24" gate="G$1" pin="P$1"/>
 <wire x1="187.96" y1="30.48" x2="187.96" y2="27.94" width="0.1524" layer="91"/>
@@
 <junction x="375.92" y="248.92"/>
 </segment>
-</net>
+<segment>
+<wire x1="157.48" y1="50.8" x2="157.48" y2="48.26" width="0.1524" layer="91"/>
+<pinref part="D5" gate="G$1" pin="C"/>
+<wire x1="149.86" y1="43.18" x2="149.86" y2="48.26" width="0.1524" layer="91"/>
+<wire x1="149.86" y1="48.26" x2="157.48" y2="48.26" width="0.1524" layer="91"/>
+<pinref part="CN3" gate="G$1" pin="P$1"/>
+<wire x1="157.48" y1="43.18" x2="157.48" y2="48.26" width="0.1524" layer="91"/>
+<junction x="157.48" y="48.26"/>
+<pinref part="VCCM8" gate="G$1" pin="VCCM"/>
+</segment>
+</net>

Commit message: initial commit
Connections:
- net GND: now also J2.1; no longer J2.4
- net VCC: now also J2.4; no longer J2.1
Other:
- note added: "addr = 0x98"
Changed lines of the file:
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@@
 <wire x1="386.08" y1="157.48" x2="421.64" y2="157.48" width="0.1524" layer="97"/>
 <text x="162.56" y="48.26" size="1.778" layer="97">to fan</text>
+<text x="190.5" y="7.62" size="2.54" layer="97" ratio="10">addr = 0x98</text>
 </plain>
 <instances>
@@
 </segment>
 <segment>
-<pinref part="J2" gate="G$1" pin="4"/>
-<wire x1="403.86" y1="167.64" x2="398.78" y2="167.64" width="0.1524" layer="91"/>
-<label x="391.16" y="167.64" size="1.778" layer="95"/>
-</segment>
-<segment>
 <pinref part="Q6" gate="G$1" pin="S"/>
 <pinref part="GND22" gate="G$1" pin="GND"/>
@@
 <wire x1="375.92" y1="241.3" x2="375.92" y2="236.22" width="0.1524" layer="91"/>
 <junction x="375.92" y="241.3"/>
+</segment>
+<segment>
+<pinref part="J2" gate="G$1" pin="1"/>
+<wire x1="403.86" y1="175.26" x2="398.78" y2="175.26" width="0.1524" layer="91"/>
+<label x="391.16" y="175.26" size="1.778" layer="95"/>
 </segment>
 </net>
@@
 </segment>
 <segment>
-<pinref part="J2" gate="G$1" pin="1"/>
-<wire x1="403.86" y1="175.26" x2="398.78" y2="175.26" width="0.1524" layer="91"/>
-<label x="391.16" y="175.26" size="1.778" layer="95"/>
-</segment>
-<segment>
 <pinref part="C24" gate="G$1" pin="P$1"/>
 <wire x1="187.96" y1="30.48" x2="187.96" y2="27.94" width="0.1524" layer="91"/>
@@
 <wire x1="203.2" y1="22.86" x2="200.66" y2="22.86" width="0.1524" layer="91"/>
 <label x="195.58" y="22.86" size="1.778" layer="95"/>
+</segment>
+<segment>
+<pinref part="J2" gate="G$1" pin="4"/>
+<wire x1="403.86" y1="167.64" x2="398.78" y2="167.64" width="0.1524" layer="91"/>
+<label x="391.16" y="167.64" size="1.778" layer="95"/>
 </segment>
 </net>
@@
 <pinref part="CONN1" gate="G$1" pin="12"/>
 <wire x1="220.98" y1="144.78" x2="223.52" y2="144.78" width="0.1524" layer="91"/>
-<label x="223.52" y="144.78" size="1.27" layer="95"/>
+<label x="223.52" y="144.78" size="1.778" layer="95"/>
 </segment>
 <segment>
@@
 <pinref part="CONN1" gate="G$1" pin="11"/>
 <wire x1="205.74" y1="144.78" x2="203.2" y2="144.78" width="0.1524" layer="91"/>
-<label x="195.58" y="144.78" size="1.27" layer="95"/>
-</segment>
-</net>
+<label x="195.58" y="144.78" size="1.778" layer="95"/>
+</segment>
+</net>

Commit message: more power
Parts:
- added C28, C29: 10u,12V, jaw:C0603
- added D6: DIODESOD-323, jaw:DIODESOD-323
- added L4, L5: (no value), jaw:L-SRR1260
- D3, D4: device jaw:DIODE-DO220AA -> jaw:DIODEDO-214AC
- L2, L3: value 220u -> 22u; device jaw:L-SRR1260 -> jaw:L2303
- Q4, Q5: value ZXMN6A08GTA -> AON6246; device jaw:MOSFET-SOT-223 -> jaw:MOSFET-DFN5X6
Connections:
- new net VIN: C1.P$1, C25.P$1, D6.C, Q2.S, R11.P$2, VREG1.VIN
- net GND: now also C28.P$2, C29.P$2
- net N$12: now also L5.P$1
- net N$2: now also L4.P$1
- net VCCM: now also C28.P$1, C29.P$1, D6.A, L4.P$2, L5.P$2; no longer C1.P$1, C25.P$1, Q2.S, R11.P$2, VREG1.VIN
Other:
- note added: "for footprint, install only one"
- moved on the sheet: C1, C25
