File: cad/ledcontrol.sch (EAGLE design)
At the start: 92 parts, among them CN1 HEADER-3X2-PTH, CN3 HEADER-1X2-THM, J1 HEADER-4X1-PTH, J2 HEADER-4X1-PTH, Q1 IRLML6344TRPBF, Q2 MOSFET-P, Q3 MOSFETSOT-23, Q4 AON6246, Q5 AON6246, Q6 IRLML6344TRPBF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

Commit message: tweak
Parts:
- C1: value .1u, 12V -> .1u, 16V
- C11, C5: value .002u -> .002u,100V
- C25, C26, C28, C29: value 10u,12V -> 10u,16V
- C27: value .1u,12V -> .1u,16V
Changed lines of the file:
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@@
 <setting verticaltext="up"/>
 </settings>
-<grid distance="0.1" unitdist="inch" unit="inch" style="lines" multiple="1" display="yes" altdistance="0.01" altunitdist="inch" altunit="inch"/>
+<grid distance="0.1" unitdist="inch" unit="inch" style="lines" multiple="1" display="no" altdistance="0.01" altunitdist="inch" altunit="inch"/>
 <layers>
-<layer number="1" name="Top" color="4" fill="1" visible="yes" active="no"/>
-<layer number="2" name="Route2" color="5" fill="1" visible="yes" active="no"/>
-<layer number="3" name="Route3" color="4" fill="3" visible="yes" active="no"/>
-<layer number="14" name="Route14" color="1" fill="6" visible="yes" active="no"/>
-<layer number="15" name="Route15" color="1" fill="1" visible="yes" active="no"/>
-<layer number="16" name="Bottom" color="6" fill="1" visible="yes" active="no"/>
-<layer number="17" name="Pads" color="2" fill="1" visible="yes" active="no"/>
-<layer number="18" name="Vias" color="2" fill="1" visible="yes" active="no"/>
-<layer number="19" name="Unrouted" color="6" fill="1" visible="yes" active="no"/>
-<layer number="20" name="Dimension" color="15" fill="1" visible="yes" active="no"/>
-<layer number="21" name="tPlace" color="7" fill="1" visible="yes" active="no"/>
-<layer number="22" name="bPlace" color="7" fill="1" visible="yes" active="no"/>
-<layer number="23" name="tOrigins" color="15" fill="1" visible="yes" active="no"/>
-<layer number="24" name="bOrigins" color="15" fill="1" visible="yes" active="no"/>
-<layer number="25" name="tNames" color="7" fill="1" visible="yes" active="no"/>
-<layer number="26" name="bNames" color="7" fill="1" visible="yes" active="no"/>
-<layer number="27" name="tValues" color="7" fill="1" visible="yes" active="no"/>
-<layer number="28" name="bValues" color="7" fill="1" visible="yes" active="no"/>
+<layer number="1" name="Top" color="4" fill="1" visible="no" active="no"/>
+<layer number="2" name="Route2" color="5" fill="1" visible="no" active="no"/>
+<layer number="3" name="Route3" color="4" fill="3" visible="no" active="no"/>
+<layer number="14" name="Route14" color="1" fill="6" visible="no" active="no"/>
+<layer number="15" name="Route15" color="1" fill="1" visible="no" active="no"/>
+<layer number="16" name="Bottom" color="6" fill="1" visible="no" active="no"/>
+<layer number="17" name="Pads" color="2" fill="1" visible="no" active="no"/>
+<layer number="18" name="Vias" color="2" fill="1" visible="no" active="no"/>
+<layer number="19" name="Unrouted" color="6" fill="1" visible="no" active="no"/>
+<layer number="20" name="Dimension" color="15" fill="1" visible="no" active="no"/>
+<layer number="21" name="tPlace" color="7" fill="1" visible="no" active="no"/>
+<layer number="22" name="bPlace" color="7" fill="1" visible="no" active="no"/>
+<layer number="23" name="tOrigins" color="15" fill="1" visible="no" active="no"/>
+<layer number="24" name="bOrigins" color="15" fill="1" visible="no" active="no"/>
+<layer number="25" name="tNames" color="7" fill="1" visible="no" active="no"/>
+<layer number="26" name="bNames" color="7" fill="1" visible="no" active="no"/>
+<layer number="27" name="tValues" color="7" fill="1" visible="no" active="no"/>
+<layer number="28" name="bValues" color="7" fill="1" visible="no" active="no"/>
 <layer number="29" name="tStop" color="7" fill="3" visible="no" active="no"/>
 <layer number="30" name="bStop" color="7" fill="6" visible="no" active="no"/>
@@
 <layer number="35" name="tGlue" color="7" fill="4" visible="no" active="no"/>
 <layer number="36" name="bGlue" color="7" fill="5" visible="no" active="no"/>
-<layer number="37" name="tTest" color="7" fill="1" visible="yes" active="no"/>
-<layer number="38" name="bTest" color="7" fill="1" visible="yes" active="no"/>
+<layer number="37" name="tTest" color="7" fill="1" visible="no" active="no"/>
+<layer number="38" name="bTest" color="7" fill="1" visible="no" active="no"/>
 <layer number="39" name="tKeepout" color="4" fill="11" visible="no" active="no"/>
 <layer number="40" name="bKeepout" color="1" fill="11" visible="no" active="no"/>
@@
 <layer number="44" name="Drills" color="7" fill="1" visible="no" active="no"/>
 <layer number="45" name="Holes" color="7" fill="1" visible="no" active="no"/>
-<layer number="46" name="Milling" color="3" fill="1" visible="yes" active="no"/>
-<layer number="47" name="Measures" color="7" fill="1" visible="yes" active="no"/>
-<layer number="48" name="Document" color="7" fill="1" visible="yes" active="no"/>
-<layer number="49" name="Reference" color="7" fill="1" visible="yes" active="no"/>
-<layer number="50" name="dxf" color="7" fill="1" visible="yes" active="no"/>
-<layer number="51" name="tDocu" color="7" fill="1" visible="yes" active="no"/>
-<layer number="52" name="bDocu" color="7" fill="1" visible="yes" active="no"/>
-<layer number="53" name="tGND_GNDA" color="7" fill="1" visible="yes" active="no"/>
-<layer number="54" name="bGND_GNDA" color="7" fill="1" visible="yes" active="no"/>
-<layer number="56" name="wert" color="7" fill="1" visible="yes" active="no"/>
-<layer number="57" name="tCAD" color="7" fill="1" visible="yes" active="no"/>
-<layer number="59" name="tCarbon" color="7" fill="1" visible="yes" active="no"/>
-<layer number="60" name="bCarbon" color="7" fill="1" visible="yes" active="no"/>
+<layer number="46" name="Milling" color="3" fill="1" visible="no" active="no"/>
+<layer number="47" name="Measures" color="7" fill="1" visible="no" active="no"/>
+<layer number="48" name="Document" color="7" fill="1" visible="no" active="no"/>
+<layer number="49" name="Reference" color="7" fill="1" visible="no" active="no"/>
+<layer number="50" name="dxf" color="7" fill="1" visible="no" active="no"/>
+<layer number="51" name="tDocu" color="7" fill="1" visible="no" active="no"/>
+<layer number="52" name="bDocu" color="7" fill="1" visible="no" active="no"/>
+<layer number="53" name="tGND_GNDA" color="7" fill="1" visible="no" active="no"/>
+<layer number="54" name="bGND_GNDA" color="7" fill="1" visible="no" active="no"/>
+<layer number="56" name="wert" color="7" fill="1" visible="no" active="no"/>
+<layer number="57" name="tCAD" color="7" fill="1" visible="no" active="no"/>
+<layer number="59" name="tCarbon" color="7" fill="1" visible="no" active="no"/>
+<layer number="60" name="bCarbon" color="7" fill="1" visible="no" active="no"/>
 <layer number="90" name="Modules" color="5" fill="1" visible="yes" active="yes"/>
 <layer number="91" name="Nets" color="2" fill="1" visible="yes" active="yes"/>
@@
 <part name="VCCM3" library="jaw" deviceset="PWR-VCCM" device=""/>
 <part name="VCC4" library="jaw" deviceset="PWR-VCC" device=""/>
-<part name="C1" library="jaw" deviceset="C" device="0603" value=".1u, 12V"/>
+<part name="C1" library="jaw" deviceset="C" device="0603" value=".1u, 16V"/>
 <part name="C2" library="jaw" deviceset="C" device="0603" value="1u"/>
 <part name="C3" library="jaw" deviceset="C" device="1210" value="100u"/>
@@
 <part name="R13" library="jaw" deviceset="R" device="0603" value="1k"/>
 <part name="R14" library="jaw" deviceset="R" device="1206" value=".01"/>
-<part name="C5" library="jaw" deviceset="C" device="0603" value=".002u"/>
+<part name="C5" library="jaw" deviceset="C" device="0603" value=".002u,100V"/>
 <part name="R15" library="jaw" deviceset="R" device="0603" value="88k7, .1%"/>
 <part name="R16" library="jaw" deviceset="R" device="0603" value="3k3, .1%"/>
@@
 <part name="R21" library="jaw" deviceset="R" device="0603" value="1k"/>
 <part name="R22" library="jaw" deviceset="R" device="1206" value=".01"/>
-<part name="C11" library="jaw" deviceset="C" device="0603" value=".002u"/>
+<part name="C11" library="jaw" deviceset="C" device="0603" value=".002u,100V"/>
 <part name="R23" library="jaw" deviceset="R" device="0603" value="88k7, .1%"/>
 <part name="R24" library="jaw" deviceset="R" device="0603" value="3k3, .1%"/>
@@
 <part name="GND23" library="jaw" deviceset="PWR-GND" device=""/>
 <part name="GND24" library="jaw" deviceset="PWR-GND" device=""/>
-<part name="C25" library="jaw" deviceset="C" device="0603" value="10u,12V"/>
-<part name="C26" library="jaw" deviceset="C" device="0603" value="10u,12V"/>
-<part name="C27" library="jaw" deviceset="C" device="0603" value=".1u,12V"/>
+<part name="C25" library="jaw" deviceset="C" device="0603" value="10u,16V"/>
+<part name="C26" library="jaw" deviceset="C" device="0603" value="10u,16V"/>
+<part name="C27" library="jaw" deviceset="C" device="0603" value=".1u,16V"/>
 <part name="VCCM7" library="jaw" deviceset="PWR-VCCM" device=""/>
 <part name="GND27" library="jaw" deviceset="PWR-GND" device=""/>
 <part name="VCCM8" library="jaw" deviceset="PWR-VCCM" device=""/>
 <part name="D6" library="jaw" deviceset="DIODE" device="SOD-323"/>
-<part name="C28" library="jaw" deviceset="C" device="0603" value="10u,12V"/>
-<part name="C29" library="jaw" deviceset="C" device="0603" value="10u,12V"/>
+<part name="C28" library="jaw" deviceset="C" device="0603" value="10u,16V"/>
+<part name="C29" library="jaw" deviceset="C" device="0603" value="10u,16V"/>
 <part name="L4" library="jaw" deviceset="L" device="-SRR1260"/>
 <part name="L5" library="jaw" deviceset="L" device="-SRR1260"/>

Commit message: more power
Parts:
- added FID1: FIDUCIALUFIDUCIAL, SparkFun-Aesthetics:FIDUCIALUFIDUCIAL
Other:
- moved on the sheet: C28, C29
Changed lines of the file:
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@@
 <part name="L4" library="jaw" deviceset="L" device="-SRR1260"/>
 <part name="L5" library="jaw" deviceset="L" device="-SRR1260"/>
+<part name="FID1" library="SparkFun-Aesthetics" deviceset="FIDUCIAL" device="UFIDUCIAL"/>
+<part name="GND28" library="jaw" deviceset="PWR-GND" device=""/>
+<part name="GND29" library="jaw" deviceset="PWR-GND" device=""/>
 </parts>
 <sheets>
@@
 <instance part="VCCM8" gate="G$1" x="157.48" y="53.34"/>
 <instance part="D6" gate="G$1" x="17.78" y="25.4"/>
-<instance part="C28" gate="G$1" x="360.68" y="243.84"/>
-<instance part="C29" gate="G$1" x="391.16" y="243.84"/>
+<instance part="C28" gate="G$1" x="287.02" y="152.4"/>
+<instance part="C29" gate="G$1" x="287.02" y="236.22"/>
 <instance part="L4" gate="G$1" x="299.72" y="236.22" rot="R90"/>
 <instance part="L5" gate="G$1" x="299.72" y="152.4" rot="R90"/>
+<instance part="FID1" gate="G$1" x="335.28" y="33.02"/>
+<instance part="GND28" gate="G$1" x="287.02" y="231.14"/>
+<instance part="GND29" gate="G$1" x="287.02" y="147.32"/>
 </instances>
 <busses>
@@
 </segment>
 <segment>
+<pinref part="C29" gate="G$1" pin="P$2"/>
+<pinref part="GND28" gate="G$1" pin="GND"/>
+</segment>
+<segment>
+<pinref part="C28" gate="G$1" pin="P$2"/>
+<pinref part="GND29" gate="G$1" pin="GND"/>
+</segment>
+<segment>
 <pinref part="C26" gate="G$1" pin="P$2"/>
 <pinref part="C27" gate="G$1" pin="P$2"/>
@@
 <wire x1="375.92" y1="241.3" x2="375.92" y2="236.22" width="0.1524" layer="91"/>
 <junction x="375.92" y="241.3"/>
-<pinref part="C28" gate="G$1" pin="P$2"/>
-<wire x1="360.68" y1="241.3" x2="370.84" y2="241.3" width="0.1524" layer="91"/>
-<junction x="370.84" y="241.3"/>
-<pinref part="C29" gate="G$1" pin="P$2"/>
-<wire x1="381" y1="241.3" x2="391.16" y2="241.3" width="0.1524" layer="91"/>
-<junction x="381" y="241.3"/>
 </segment>
 <segment>
@@
 </segment>
 <segment>
+<pinref part="R17" gate="G$1" pin="P$2"/>
+<pinref part="VCCM5" gate="G$1" pin="VCCM"/>
+</segment>
+<segment>
+<pinref part="CONN1" gate="G$1" pin="12"/>
+<wire x1="220.98" y1="144.78" x2="223.52" y2="144.78" width="0.1524" layer="91"/>
+<label x="223.52" y="144.78" size="1.778" layer="95"/>
+</segment>
+<segment>
 <pinref part="L2" gate="G$1" pin="P$2"/>
 <pinref part="VCCM4" gate="G$1" pin="VCCM"/>
+<junction x="307.34" y="243.84"/>
 <pinref part="L4" gate="G$1" pin="P$2"/>
 <wire x1="299.72" y1="243.84" x2="307.34" y2="243.84" width="0.1524" layer="91"/>
-<junction x="307.34" y="243.84"/>
-</segment>
-<segment>
-<pinref part="R17" gate="G$1" pin="P$2"/>
-<pinref part="VCCM5" gate="G$1" pin="VCCM"/>
-</segment>
-<segment>
+<junction x="299.72" y="243.84"/>
+<wire x1="287.02" y1="243.84" x2="299.72" y2="243.84" width="0.1524" layer="91"/>
+<pinref part="C29" gate="G$1" pin="P$1"/>
+<wire x1="287.02" y1="241.3" x2="287.02" y2="243.84" width="0.1524" layer="91"/>
+</segment>
+<segment>
+<pinref part="VCCM7" gate="G$1" pin="VCCM"/>
+<pinref part="C27" gate="G$1" pin="P$1"/>
+<wire x1="375.92" y1="248.92" x2="381" y2="248.92" width="0.1524" layer="91"/>
+<wire x1="375.92" y1="248.92" x2="375.92" y2="251.46" width="0.1524" layer="91"/>
+<junction x="375.92" y="248.92"/>
+<pinref part="C26" gate="G$1" pin="P$1"/>
+<wire x1="370.84" y1="248.92" x2="375.92" y2="248.92" width="0.1524" layer="91"/>
+</segment>
+<segment>
+<pinref part="C28" gate="G$1" pin="P$1"/>
 <pinref part="L3" gate="G$1" pin="P$2"/>
 <pinref part="VCCM6" gate="G$1" pin="VCCM"/>
@@
 <wire x1="299.72" y1="160.02" x2="307.34" y2="160.02" width="0.1524" layer="91"/>
 <junction x="307.34" y="160.02"/>
-</segment>
-<segment>
-<pinref part="CONN1" gate="G$1" pin="12"/>
-<wire x1="220.98" y1="144.78" x2="223.52" y2="144.78" width="0.1524" layer="91"/>
-<label x="223.52" y="144.78" size="1.778" layer="95"/>
-</segment>
-<segment>
-<pinref part="C26" gate="G$1" pin="P$1"/>
-<pinref part="C27" gate="G$1" pin="P$1"/>
-<wire x1="370.84" y1="248.92" x2="375.92" y2="248.92" width="0.1524" layer="91"/>
-<pinref part="VCCM7" gate="G$1" pin="VCCM"/>
-<wire x1="375.92" y1="248.92" x2="381" y2="248.92" width="0.1524" layer="91"/>
-<wire x1="375.92" y1="248.92" x2="375.92" y2="251.46" width="0.1524" layer="91"/>
-<junction x="375.92" y="248.92"/>
-<pinref part="C29" gate="G$1" pin="P$1"/>
-<wire x1="391.16" y1="248.92" x2="381" y2="248.92" width="0.1524" layer="91"/>
-<junction x="381" y="248.92"/>
-<pinref part="C28" gate="G$1" pin="P$1"/>
-<wire x1="370.84" y1="248.92" x2="360.68" y2="248.92" width="0.1524" layer="91"/>
-<junction x="370.84" y="248.92"/>
-</segment>
-<segment>
+<wire x1="287.02" y1="157.48" x2="287.02" y2="160.02" width="0.1524" layer="91"/>
+<wire x1="287.02" y1="160.02" x2="299.72" y2="160.02" width="0.1524" layer="91"/>
+<junction x="299.72" y="160.02"/>
+</segment>
+<segment>
